File: Adafruit Circuit Playground TFT Gizmo.sch (EAGLE design)
At the start: 43 parts, among them IC4 APX803-SAG, Q1 BSS138, U5 PAM8302AASCR

Commit message: Updated to D1 Revision
Connections:
- net A1' renamed A1_
- net A2' renamed A2_
Other:
- note added: "Backlight"
- note added: "JST Connectors"
- note added: "Reset"
- note added: "Test Points"
- note removed: "Slide Switch"
- moved on the sheet: C1, C13, C15, C2, C9, D1, D2, IC4, LEFT, Q1, R1, R12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
